File: tpa3116_amplifier_board_pbtl_mono.kicad_pcb (KiCad board)
At the start: 2 copper layers, 59.7 x 50.8 mm, 47 parts, among them IC1 TPA3116D2QDADRQ1, J1 power_supply, J2 Conn_01x04, J3 power_supply, J4 output_right

Commit message: Убрал лишние переходные отверстия, изображение обновил
Routing:
- net GND: vias 96 -> 80
Changed lines of the file:
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@@
+  )
+  (dimension (type aligned) (layer "Dwgs.User")
+    (pts (xy 124.46 100) (xy 124.46 140))
+    (height 28.575)
+    (gr_text "40,0000 mm" (at 94.735 120 90) (layer "Dwgs.User")
+      (effects (font (size 1 1) (thickness 0.15)))
+    )
+    (format (prefix "") (suffix "") (units 3) (units_format 1) (precision 4))
+    (style (thickness 0.1) (arrow_length 1.27) (text_position_mode 0) (extension_height 0.58642) (extension_offset 0.5) keep_text_aligned)
   )
   (dimension (type aligned) (layer "Dwgs.User")
@@
   (via (at 147.955 118.11) (size 0.8) (drill 0.4) (layers "F.Cu" "B.Cu") (free) (net 5))
   (via (at 125.73 125.095) (size 0.8) (drill 0.4) (layers "F.Cu" "B.Cu") (free) (net 5))
-  (via (at 110.49 123.825) (size 0.8) (drill 0.4) (layers "F.Cu" "B.Cu") (free) (net 5))
-  (via (at 145.415 121.92) (size 0.8) (drill 0.4) (layers "F.Cu" "B.Cu") (free) (net 5))
-  (via (at 142.875 129.54) (size 0.8) (drill 0.4) (layers "F.Cu" "B.Cu") (free) (net 5))
+  (via (at 109.855 123.825) (size 0.8) (drill 0.4) (layers "F.Cu" "B.Cu") (free) (net 5))
+  (via (at 142.875 132.08) (size 0.8) (drill 0.4) (layers "F.Cu" "B.Cu") (free) (net 5))
   (via (at 156.845 121.92) (size 0.8) (drill 0.4) (layers "F.Cu" "B.Cu") (free) (net 5))
   (via (at 147.955 107.95) (size 0.8) (drill 0.4) (layers "F.Cu" "B.Cu") (free) (net 5))
@@
   (via (at 123.19 114.935) (size 0.8) (drill 0.4) (layers "F.Cu" "B.Cu") (free) (net 5))
   (via (at 137.665 121.92) (size 0.8) (drill 0.4) (layers "F.Cu" "B.Cu") (free) (net 5))
-  (via (at 109.22 123.825) (size 0.8) (drill 0.4) (layers "F.Cu" "B.Cu") (free) (net 5))
+  (via (at 111.125 123.825) (size 0.8) (drill 0.4) (layers "F.Cu" "B.Cu") (free) (net 5))
   (via (at 122.533 109.855) (size 0.8) (drill 0.4) (layers "F.Cu" "B.Cu") (free) (net 5))
   (via (at 122.555 133.985) (size 0.8) (drill 0.4) (layers "F.Cu" "B.Cu") (free) (net 5))
-  (via (at 145.415 132.08) (size 0.8) (drill 0.4) (layers "F.Cu" "B.Cu") (free) (net 5))
+  (via (at 151.13 139.7) (size 0.8) (drill 0.4) (layers "F.Cu" "B.Cu") (free) (net 5))
   (via (at 110.49 117.475) (size 0.8) (drill 0.4) (layers "F.Cu" "B.Cu") (free) (net 5))
   (via (at 151.13 105.41) (size 0.8) (drill 0.4) (layers "F.Cu" "B.Cu") (free) (net 5))
@@
   (via (at 113.665 110.49) (size 0.8) (drill 0.4) (layers "F.Cu" "B.Cu") (free) (net 5))
   (via (at 123.825 107.315) (size 0.8) (drill 0.4) (layers "F.Cu" "B.Cu") (free) (net 5))
-  (via (at 121.263 129.54) (size 0.8) (drill 0.4) (layers "F.Cu" "B.Cu") (free) (net 5))
   (via (at 124.46 123.825) (size 0.8) (drill 0.4) (layers "F.Cu" "B.Cu") (free) (net 5))
   (via (at 154.94 120.015) (size 0.8) (drill 0.4) (layers "F.Cu" "B.Cu") (free) (net 5))
+  (via (at 147.955 134.62) (size 0.8) (drill 0.4) (layers "F.Cu" "B.Cu") (free) (net 5))
   (via (at 156.845 120.015) (size 0.8) (drill 0.4) (layers "F.Cu" "B.Cu") (free) (net 5))
   (via (at 111.76 117.475) (size 0.8) (drill 0.4) (layers "F.Cu" "B.Cu") (free) (net 5))
   (via (at 151.13 102.87) (size 0.8) (drill 0.4) (layers "F.Cu" "B.Cu") (free) (net 5))
   (via (at 124.46 116.205) (size 0.8) (drill 0.4) (layers "F.Cu" "B.Cu") (free) (net 5))
+  (via (at 147.955 105.41) (size 0.8) (drill 0.4) (layers "F.Cu" "B.Cu") (free) (net 5))
   (via (at 147.955 120.015) (size 0.8) (drill 0.4) (layers "F.Cu" "B.Cu") (free) (net 5))
   (via (at 129.54 142.875) (size 0.8) (drill 0.4) (layers "F.Cu" "B.Cu") (free) (net 5))
@@
   (via (at 122.533 128.905) (size 0.8) (drill 0.4) (layers "F.Cu" "B.Cu") (free) (net 5))
   (via (at 119.38 97.155) (size 0.8) (drill 0.4) (layers "F.Cu" "B.Cu") (free) (net 5))
-  (via (at 147.955 137.16) (size 0.8) (drill 0.4) (layers "F.Cu" "B.Cu") (free) (net 5))
-  (via (at 121.285 111.76) (size 0.8) (drill 0.4) (layers "F.Cu" "B.Cu") (free) (net 5))
   (via (at 124.46 125.095) (size 0.8) (drill 0.4) (layers "F.Cu" "B.Cu") (free) (net 5))
   (via (at 126.365 107.315) (size 0.8) (drill 0.4) (layers "F.Cu" "B.Cu") (free) (net 5))
-  (via (at 111.76 123.825) (size 0.8) (drill 0.4) (layers "F.Cu" "B.Cu") (free) (net 5))
-  (via (at 140.97 118.11) (size 0.8) (drill 0.4) (layers "F.Cu" "B.Cu") (free) (net 5))
   (via (at 156.21 137.16) (size 0.8) (drill 0.4) (layers "F.Cu" "B.Cu") (free) (net 5))
   (via (at 124.46 117.475) (size 0.8) (drill 0.4) (layers "F.Cu" "B.Cu") (free) (net 5))
   (via (at 147.955 121.92) (size 0.8) (drill 0.4) (layers "F.Cu" "B.Cu") (free) (net 5))
   (via (at 114.3 102.235) (size 0.8) (drill 0.4) (layers "F.Cu" "B.Cu") (free) (net 5))
-  (via (at 142.875 110.49) (size 0.8) (drill 0.4) (layers "F.Cu" "B.Cu") (free) (net 5))
-  (via (at 147.955 134.62) (size 0.8) (drill 0.4) (layers "F.Cu" "B.Cu") (free) (net 5))
+  (via (at 142.875 107.95) (size 0.8) (drill 0.4) (layers "F.Cu" "B.Cu") (free) (net 5))
   (via (at 147.955 132.08) (size 0.8) (drill 0.4) (layers "F.Cu" "B.Cu") (free) (net 5))
-  (via (at 121.263 127) (size 0.8) (drill 0.4) (layers "F.Cu" "B.Cu") (free) (net 5))
-  (via (at 147.955 102.87) (size 0.8) (drill 0.4) (layers "F.Cu" "B.Cu") (free) (net 5))
   (via (at 129.54 102.235) (size 0.8) (drill 0.4) (layers "F.Cu" "B.Cu") (free) (net 5))
   (via (at 122.533 111.125) (size 0.8) (drill 0.4) (layers "F.Cu" "B.Cu") (free) (net 5))
-  (via (at 145.415 120.015) (size 0.8) (drill 0.4) (layers "F.Cu" "B.Cu") (free) (net 5))
+  (via (at 149.86 120.015) (size 0.8) (drill 0.4) (layers "F.Cu" "B.Cu") (free) (net 5))
   (via (at 114.935 142.875) (size 0.8) (drill 0.4) (layers "F.Cu" "B.Cu") (free) (net 5))
   (via (at 156.845 123.825) (size 0.8) (drill 0.4) (layers "F.Cu" "B.Cu") (free) (net 5))
-  (via (at 140.335 107.95) (size 0.8) (drill 0.4) (layers "F.Cu" "B.Cu") (free) (net 5))
-  (via (at 121.263 128.27) (size 0.8) (drill 0.4) (layers "F.Cu" "B.Cu") (free) (net 5))
+  (via (at 137.795 107.95) (size 0.8) (drill 0.4) (layers "F.Cu" "B.Cu") (free) (net 5))
   (via (at 151.13 137.16) (size 0.8) (drill 0.4) (layers "F.Cu" "B.Cu") (free) (net 5))
-  (via (at 140.97 121.92) (size 0.8) (drill 0.4) (layers "F.Cu" "B.Cu") (free) (net 5))
-  (via (at 151.13 139.7) (size 0.8) (drill 0.4) (layers "F.Cu" "B.Cu") (free) (net 5))
-  (via (at 142.875 115.57) (size 0.8) (drill 0.4) (layers "F.Cu" "B.Cu") (free) (net 5))
   (via (at 156.845 118.11) (size 0.8) (drill 0.4) (layers "F.Cu" "B.Cu") (free) (net 5))
-  (via (at 145.415 118.11) (size 0.8) (drill 0.4) (layers "F.Cu" "B.Cu") (free) (net 5))
   (via (at 156.21 102.87) (size 0.8) (drill 0.4) (layers "F.Cu" "B.Cu") (free) (net 5))
   (via (at 125.73 116.205) (size 0.8) (drill 0.4) (layers "F.Cu" "B.Cu") (free) (net 5))
@@
   (via (at 123.19 122.555) (size 0.8) (drill 0.4) (layers "F.Cu" "B.Cu") (free) (net 5))
   (via (at 125.73 114.935) (size 0.8) (drill 0.4) (layers "F.Cu" "B.Cu") (free) (net 5))
+  (via (at 142.875 118.11) (size 0.8) (drill 0.4) (layers "F.Cu" "B.Cu") (free) (net 5))
+  (via (at 142.875 121.92) (size 0.8) (drill 0.4) (layers "F.Cu" "B.Cu") (free) (net 5))
   (via (at 134.62 97.155) (size 0.8) (drill 0.4) (layers "F.Cu" "B.Cu") (free) (net 5))
-  (via (at 142.875 124.46) (size 0.8) (drill 0.4) (layers "F.Cu" "B.Cu") (free) (net 5))
-  (via (at 147.955 105.41) (size 0.8) (drill 0.4) (layers "F.Cu" "B.Cu") (free) (net 5))
   (via (at 123.19 123.825) (size 0.8) (drill 0.4) (layers "F.Cu" "B.Cu") (free) (net 5))
   (via (at 116.205 129.54) (size 0.8) (drill 0.4) (layers "F.Cu" "B.Cu") (free) (net 5))
-  (via (at 121.285 113.03) (size 0.8) (drill 0.4) (layers "F.Cu" "B.Cu") (free) (net 5))
-  (via (at 119.38 102.235) (size 0.8) (drill 0.4) (layers "F.Cu" "B.Cu") (free) (net 5))
   (via (at 109.22 117.475) (size 0.8) (drill 0.4) (layers "F.Cu" "B.Cu") (free) (net 5))
   (via (at 116.205 127) (size 0.8) (drill 0.4) (layers "F.Cu" "B.Cu") (free) (net 5))
@@
   (via (at 119.38 142.875) (size 0.8) (drill 0.4) (layers "F.Cu" "B.Cu") (free) (net 5))
   (via (at 114.935 137.795) (size 0.8) (drill 0.4) (layers "F.Cu" "B.Cu") (free) (net 5))
-  (via (at 145.415 107.95) (size 0.8) (drill 0.4) (layers "F.Cu" "B.Cu") (free) (net 5))
   (via (at 124.46 114.935) (size 0.8) (drill 0.4) (layers "F.Cu" "B.Cu") (free) (net 5))
   (via (at 123.19 116.205) (size 0.8) (drill 0.4) (layers "F.Cu" "B.Cu") (free) (net 5))
@@
   (via (at 122.533 126.365) (size 0.8) (drill 0.4) (layers "F.Cu" "B.Cu") (free) (net 5))
   (via (at 122.533 127.635) (size 0.8) (drill 0.4) (layers "F.Cu" "B.Cu") (free) (net 5))
-  (via (at 121.285 110.49) (size 0.8) (drill 0.4) (layers "F.Cu" "B.Cu") (free) (net 5))
   (via (at 129.54 137.795) (size 0.8) (drill 0.4) (layers "F.Cu" "B.Cu") (free) (net 5))
   (via (at 125.73 117.475) (size 0.8) (drill 0.4) (layers "F.Cu" "B.Cu") (free) (net 5))
-  (via (at 140.335 132.08) (size 0.8) (drill 0.4) (layers "F.Cu" "B.Cu") (free) (net 5))
+  (via (at 137.795 132.08) (size 0.8) (drill 0.4) (layers "F.Cu" "B.Cu") (free) (net 5))
   (via (at 122.555 130.175) (size 0.8) (drill 0.4) (layers "F.Cu" "B.Cu") (free) (net 5))
   (via (at 163.195 102.87) (size 0.8) (drill 0.4) (layers "F.Cu" "B.Cu") (free) (net 5))
